File: saha-aux.brd (EAGLE design)
At the start: 100 x 56 mm, 74 parts, among them K1 EC2-5NU, K2 EC2-5NU, K3 EC2-5NU, K4 EC2-5NU, X1 S4B-PH-SM4-TB, X2 S4B-PH-SM4-TB, X3 EBWA-03-B, X4 EBWA-03-B, X5 EBWA-03-B, X6 S8B-PH-SM4-TB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

Commit message: placement round 1
Parts:
- removed LED1, LED2, LED3, LED4: (no value), saha-aux:CHIP-LED0603
- added H1, H2, H3, H4: LED-GRN, saha-aux:CHIP-LED0603
- added V10, V11, V12, V9: MMDL914, saha-aux:SOD-323
- moved R17 268.7 mm to (68.8, 38.2), turned to 90 degrees
- moved R16 258.6 mm to (72.2, 31.0), turned to 180 degrees
- moved R18 258.5 mm to (76.2, 33.2), turned to 180 degrees
- moved K4 258.0 mm to (71.8, 38.0)
- moved V7 256.4 mm to (72.2, 34.0)
- moved R15 253.5 mm to (58.2, 33.2), turned to 180 degrees
- moved R13 253.3 mm to (54.0, 31.0), turned to 180 degrees
- moved C11 252.6 mm to (68.8, 31.0)
- moved V8 251.9 mm to (68.8, 34.0)
- moved V6 251.6 mm to (50.5, 34.0)
- moved C10 249.9 mm to (50.5, 31.0)
- moved R14 247.4 mm to (50.5, 38.2), turned to 90 degrees
- moved X7 246.2 mm to (75.8, 51.0)
- moved X5 244.3 mm to (57.5, 51.0)
- moved K3 241.9 mm to (53.5, 38.0)
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Connections:
- net N$1 renamed A0
- net N$2 renamed A1
- net N$3 renamed A2
- net N$4 renamed RESET_N
- removed net N$10: K1.12, R8.2, V1.3
- removed net N$16: K2.12, R11.2, V3.3
- removed net N$23: K3.12, R14.2, V5.3
- removed net N$30: K4.12, R17.2, V7.3
- new net +5V1: K2.1, V10.C
- new net +5V2: K3.1, V11.C
- new net COILN1: K1.12, R8.2, V1.3, V9.A
- new net COILN2: K2.12, R11.2, V10.A, V3.3
- new net COILN3: K3.12, R14.2, V11.A, V5.3
- new net COILN4: K4.12, R17.2, V12.A, V7.3
- net +5V: now also V12.C, V9.C; no longer K2.1, K3.1
- net GND: now also H1.C, H2.C, H3.C, H4.C; no longer LED1.C, LED2.C, LED3.C, LED4.C
- net N$18: now also H2.A; no longer LED2.A
- net N$25: now also H3.A; no longer LED3.A
- net N$32: now also H4.A; no longer LED4.A
- net N$6: now also H1.A; no longer LED1.A
- net RELAY_1: now also D3.14; no longer D3.11
- net RELAY_2: now also D3.13; no longer D3.12
- net RELAY_3: now also D3.12; no longer D3.13
- net RELAY_4: now also D3.11; no longer D3.14
Routing:
- net +5V: track 112.1 -> 0.00 mm, vias 2 -> 0
- net I2CSCL: track 90.8 -> 0.00 mm, vias 3 -> 0
- net I2CSDA: track 90.5 -> 0.00 mm, vias 3 -> 0
- net GND: track 7.42 -> 0.00 mm, vias 23 -> 0

Commit message: finished v1.00
Parts:
- added C12, C13: 22u, saha-aux:C0805
- added R19, R20, R21: 0R0, saha-aux:R0603
- C3: value 100n -> 22u; device saha-aux:C0603 -> saha-aux:C0805
- X6: value S8B-PH-SM4-TB -> EBWA-03-B; device saha-cpu:JST-PH2.0-RA-8 -> saha-aux:RUUVILIITIN381-3
- X7: value EBWA-03-B -> S8B-PH-SM4-TB; device saha-aux:RUUVILIITIN381-3 -> saha-cpu:JST-PH2.0-RA-8
- moved U$1 68.2 mm to (66.8, 8.75)
- moved C3 58.7 mm to (5.75, 15.8), turned to 180 degrees
- moved X7 56.2 mm to (50.0, 1.00), turned to 180 degrees
- moved X6 56.1 mm to (75.5, 51.0), turned to 0 degrees
- moved C1 52.5 mm to (9.35, 39.5), turned to 90 degrees
- moved C2 26.7 mm to (88.2, 20.8)
- moved D4 16.2 mm to (35.0, 25.5), turned to 180 degrees
- moved C7 15.9 mm to (32.2, 26.0), turned to 90 degrees
- moved R6 15.2 mm to (37.8, 26.0), turned to 270 degrees
- moved R5 7.83 mm to (32.0, 17.2), turned to 180 degrees
- moved R4 5.52 mm to (36.5, 17.2), turned to 0 degrees
- moved R3 2.75 mm to (20.2, 4.25), turned to 90 degrees
- moved R2 2.00 mm to (18.5, 4.25), turned to 90 degrees
- moved C4 1.68 mm to (20.5, 14.5), turned to 180 degrees
- moved C5 1.58 mm to (30.5, 14.5), turned to 180 degrees
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Connections:
- net N$12 renamed NC2
- net N$13 renamed NO2
- net N$14 renamed COM2
- net N$19 renamed NC3
- net N$20 renamed NO3
- net N$21 renamed COM3
- net N$5 renamed NC1
- net N$7 renamed NO1
- net N$8 renamed COM1
- removed net +5V1: K2.1, V10.C
- removed net +5V2: K3.1, V11.C
- removed net N$26: K4.10, K4.3, X7.1
- removed net N$27: K4.5, K4.8, X7.3
- removed net N$28: K4.4, K4.9, X7.2
- new net COM4: K4.4, K4.9, X6.2
- new net NC4: K4.10, K4.3, X6.1
- new net NO4: K4.5, K4.8, X6.3
- net +5V: now also C12.1, C13.1, K2.1, K3.1, V10.C, V11.C
- net A0: now also R19.2
- net A1: now also R20.2
- net A2: now also R21.2
- net GND: now also C12.2, C13.2, R19.1, R20.1, R21.1, X7.2, X7.4, X7.6, X7.8; no longer X6.2, X6.4, X6.6, X6.8
- net IN1: now also X7.1; no longer X6.1
- net IN2: now also X7.3; no longer X6.3
- net IN3: now also X7.5; no longer X6.5
- net IN4: now also X7.7; no longer X6.7
Routing:
- net +5V: track 0.00 -> 316.6 mm, vias 0 -> 17
- net I2CSDA: track 0.00 -> 128.7 mm, vias 0 -> 4
- net I2CSCL: track 0.00 -> 120.6 mm, vias 0 -> 4
- net A0: track 0.00 -> 45.2 mm, vias 0 -> 2
- net A1: track 0.00 -> 44.9 mm, vias 0 -> 2
- net A2: track 0.00 -> 43.7 mm, vias 0 -> 2
- net RELAY_1: track 0.00 -> 43.3 mm
- net RELAY_4: track 0.00 -> 32.0 mm
- net RELAY_2: track 0.00 -> 26.6 mm
- net IN4_F: track 0.00 -> 20.9 mm
- net RELAY_3: track 0.00 -> 16.5 mm
- net IN3_F: track 0.00 -> 16.4 mm
- net IN1_F: track 0.00 -> 15.2 mm
- net GND: track 0.00 -> 14.0 mm, vias 0 -> 72
- net NC4: track 0.00 -> 13.6 mm
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Other:
- board text added: "#1"
- board text added: "#2"
- board text added: "#3"
- board text added: "#4"
- board text added: "A0 A1 A2"
- board text added: "NC"
- board text added: "NO"
- board text added: "SAHA AUX V1.00"

Commit message: remove bottom silk
Parts:
- removed U$3: DAFUG, saha-aux:DAFUG
Other:
- board text removed: "+5V SDA GND SCL"
- board text removed: "A B C"
- board text removed: "I2C ADDRESS 0x70...0x77 1110ABC"
- board text removed: "KS0 KS1 KS2 K4 K3 K2 K1 K0"
- board text removed: "SAHA DISPLAY V1.0"
- board text removed: "SCL GND SDA +5V"
Changed lines of the file:
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@@
 <layer number="20" name="Dimension" color="24" fill="1" visible="yes" active="yes"/>
 <layer number="21" name="tPlace" color="7" fill="1" visible="yes" active="yes"/>
-<layer number="22" name="bPlace" color="7" fill="1" visible="no" active="yes"/>
+<layer number="22" name="bPlace" color="7" fill="1" visible="yes" active="yes"/>
 <layer number="23" name="tOrigins" color="15" fill="1" visible="yes" active="yes"/>
 <layer number="24" name="bOrigins" color="15" fill="1" visible="yes" active="yes"/>
@@
 <dimension x1="3.5" y1="52.5" x2="96.5" y2="52.5" x3="50" y3="62" textsize="2.5" layer="47" dtype="horizontal"/>
 <dimension x1="96.5" y1="52.5" x2="96.5" y2="3.5" x3="116.9" y3="28" textsize="2.5" layer="47" dtype="vertical"/>
-<text x="81.2" y="34.5" size="1.5" layer="22" font="vector" rot="MR0">I2C ADDRESS
-0x70...0x77
-1110ABC</text>
-<text x="65.6" y="37.5" size="1.7" layer="22" font="vector" distance="22" rot="MR0" align="center-left">A
-B
-C</text>
-<text x="77.2" y="50.9" size="2.5" layer="22" font="vector" rot="MR0">KIMMOLI 2019</text>
-<text x="46.7" y="51" size="2.5" layer="22" font="vector" rot="MR0">SAHA DISPLAY V1.0</text>
-<text x="87.9" y="28" size="1.4" layer="22" font="vector" distance="45" rot="MR0" align="center-left">+5V
-SDA
-GND
-SCL</text>
-<text x="12.7" y="28" size="1.4" layer="22" font="vector" distance="45" rot="MR0" align="center-right">SCL
-GND
-SDA
-+5V</text>
-<text x="50.1" y="11.8" size="1.4" layer="22" font="vector" distance="45" rot="SMR90" align="center-left">KS0
-KS1
-KS2
-K4
-K3
-K2
-K1
-K0</text>
 <text x="86" y="1.6" size="2" layer="1" font="vector" ratio="12" align="center-left">1  </text>
 <text x="89" y="1.6" size="2" layer="16" font="vector" ratio="12" rot="MR0" align="center-left">2</text>
@@
 </element>
 <element name="U$1" library="saha-aux" package="DAFUG" value="DAFUG" x="66.75" y="8.75" smashed="yes"/>
-<element name="U$3" library="saha-aux" package="DAFUG" value="DAFUG" x="87.05" y="52" smashed="yes" rot="MR0"/>
 <element name="D1" library="saha-aux" package="SOIC8-N" value="LM75BD" x="19" y="11" smashed="yes">
 <attribute name="NAME" x="17.2474" y="13.794" size="0.9" layer="25" font="vector" ratio="10" rot="SR0"/>
