File: saha-aux.sch (EAGLE design)
At the start: 73 parts, among them K1 EC2-5NU, K2 EC2-5NU, K3 EC2-5NU, K4 EC2-5NU, X1 S4B-PH-SM4-TB, X2 S4B-PH-SM4-TB, X3 EBWA-03-B, X4 EBWA-03-B, X5 EBWA-03-B, X6 S8B-PH-SM4-TB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

Commit message: placement round 1
Parts:
- removed LED1, LED2, LED3, LED4: (no value), saha-aux:LEDCHIP-LED0603
- added H1, H2, H3, H4: LED-GRN, saha-aux:LED-GRN
- added V10, V11, V12, V9: MMDL914, saha-aux:MMDL914
Connections:
- net N$1 renamed A0
- net N$2 renamed A1
- net N$3 renamed A2
- net N$4 renamed RESET_N
- removed net N$10: K1.COILN, R8.2, V1.D
- removed net N$16: K2.COILN, R11.2, V3.D
- removed net N$23: K3.COILN, R14.2, V5.D
- removed net N$30: K4.COILN, R17.2, V7.D
- new net +5V1: K2.COILP, V10.C
- new net +5V2: K3.COILP, V11.C
- new net COILN1: K1.COILN, R8.2, V1.D, V9.A
- new net COILN2: K2.COILN, R11.2, V10.A, V3.D
- new net COILN3: K3.COILN, R14.2, V11.A, V5.D
- new net COILN4: K4.COILN, R17.2, V12.A, V7.D
- net +5V: now also V12.C, V9.C; no longer K2.COILP, K3.COILP
- net GND: now also H1.C, H2.C, H3.C, H4.C; no longer LED1.C, LED2.C, LED3.C, LED4.C
- net N$18: now also H2.A; no longer LED2.A
- net N$25: now also H3.A; no longer LED3.A
- net N$32: now also H4.A; no longer LED4.A
- net N$6: now also H1.A; no longer LED1.A
- net RELAY_1: now also D3.P7; no longer D3.P4
- net RELAY_2: now also D3.P6; no longer D3.P5
- net RELAY_3: now also D3.P5; no longer D3.P6
- net RELAY_4: now also D3.P4; no longer D3.P7

Commit message: finished v1.00
Parts:
- added C12, C13: 22u, saha-aux:CAP0805
- added R19, R20, R21: 0R0, saha-aux:RES0603
- C3: value 100n -> 22u; device saha-aux:CAP0603 -> saha-aux:CAP0805
- X6: value S8B-PH-SM4-TB -> EBWA-03-B; device saha-cpu:S8B-PH-SM4-TB -> saha-aux:EBWA-03-B
- X7: value EBWA-03-B -> S8B-PH-SM4-TB; device saha-aux:EBWA-03-B -> saha-cpu:S8B-PH-SM4-TB
Connections:
- net N$12 renamed NC2
- net N$13 renamed NO2
- net N$14 renamed COM2
- net N$19 renamed NC3
- net N$20 renamed NO3
- net N$21 renamed COM3
- net N$5 renamed NC1
- net N$7 renamed NO1
- net N$8 renamed COM1
- removed net +5V1: K2.COILP, V10.C
- removed net +5V2: K3.COILP, V11.C
- removed net N$26: K4.NC1, K4.NC2, X7.1
- removed net N$27: K4.NO1, K4.NO2, X7.3
- removed net N$28: K4.COM1, K4.COM2, X7.2
- new net COM4: K4.COM1, K4.COM2, X6.2
- new net NC4: K4.NC1, K4.NC2, X6.1
- new net NO4: K4.NO1, K4.NO2, X6.3
- net +5V: now also C12.1, C13.1, K2.COILP, K3.COILP, V10.C, V11.C
- net A0: now also R19.2
- net A1: now also R20.2
- net A2: now also R21.2
- net GND: now also C12.2, C13.2, R19.1, R20.1, R21.1, X7.2, X7.4, X7.6, X7.8; no longer X6.2, X6.4, X6.6, X6.8
- net IN1: now also X7.1; no longer X6.1
- net IN2: now also X7.3; no longer X6.3
- net IN3: now also X7.5; no longer X6.5
- net IN4: now also X7.7; no longer X6.7
Other:
- note added: "0x48..0x4F 0x18..0x1F 0x50..0x57"
- note added: "LM75 PCA9557DR 24C64"
